File: 555/555.kicad_sch (KiCad schematic)
At the start: 10 parts, among them U1 LM555xM, U2 TSOP17xx

Commit message: 555 actualizada
Parts:
- C1: renamed from C2; footprint (none) -> Capacitor_THT:C_Disc_D4.3mm_W1.9mm_P5.00mm
- C2: renamed from C1; footprint (none) -> Capacitor_THT:C_Disc_D4.3mm_W1.9mm_P5.00mm
- D1: footprint (none) -> LED_THT:LED_D5.0mm_Horizontal_O1.27mm_Z3.0mm
- R1: renamed from R3; footprint (none) -> Resistor_THT:R_Axial_DIN0204_L3.6mm_D1.6mm_P5.08mm_Horizontal
- R2, R4: footprint (none) -> Resistor_THT:R_Axial_DIN0204_L3.6mm_D1.6mm_P2.54mm_Vertical
- R3: renamed from R1; footprint (none) -> Resistor_THT:R_Axial_DIN0204_L3.6mm_D1.6mm_P2.54mm_Vertical
- RV1: footprint (none) -> Potentiometer_THT:Potentiometer_Bourns_3296W_Vertical
- U1: footprint Package_SO:SOIC-8_3.9x4.9mm_P1.27mm -> Package_DIP:DIP-8_W7.62mm
- U2: footprint OptoDevice:Vishay_CAST-3Pin -> Package_TO_SOT_THT:TO-92S_Wide
Changed lines of the file:
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@@
   (junction (at 53.34 85.09) (diameter 0) (color 0 0 0 0)
   )
-  (junction (at 57.15 27.94) (diameter 0) (color 0 0 0 0)
+  (junction (at 63.5 27.94) (diameter 0) (color 0 0 0 0)
   )
   (junction (at 66.04 33.02) (diameter 0) (color 0 0 0 0)
@@
     (stroke (width 0) (type default))
   )
-  (wire (pts (xy 57.15 41.91) (xy 57.15 38.1))
-    (stroke (width 0) (type default))
-  )
   (wire (pts (xy 53.34 74.93) (xy 66.04 74.93))
     (stroke (width 0) (type default))
@@
     (stroke (width 0) (type default))
   )
+  (wire (pts (xy 57.15 38.1) (xy 57.15 41.91))
+    (stroke (width 0) (type default))
+  )
   (wire (pts (xy 27.94 41.91) (xy 27.94 36.83))
     (stroke (width 0) (type default))
   )
-  (wire (pts (xy 57.15 24.13) (xy 57.15 27.94))
-    (stroke (width 0) (type default))
-  )
-  (wire (pts (xy 57.15 24.13) (xy 27.94 24.13))
+  (wire (pts (xy 63.5 24.13) (xy 63.5 27.94))
+    (stroke (width 0) (type default))
+  )
+  (wire (pts (xy 63.5 24.13) (xy 27.94 24.13))
     (stroke (width 0) (type default))
   )
@@
     (stroke (width 0) (type default))
   )
+  (wire (pts (xy 63.5 27.94) (xy 67.31 27.94))
+    (stroke (width 0) (type default))
+  )
   (wire (pts (xy 57.15 33.02) (xy 66.04 33.02))
     (stroke (width 0) (type default))
@@
     (stroke (width 0) (type default))
   )
-  (wire (pts (xy 57.15 27.94) (xy 67.31 27.94))
+  (wire (pts (xy 57.15 27.94) (xy 63.5 27.94))
     (stroke (width 0) (type default))
   )
@@
   (symbol (lib_id "Device:C") (at 27.94 33.02 0) (unit 1)
     (in_bom yes) (on_board yes) (dnp no) (fields_autoplaced)
-    (property "Reference" "C1" (at 31.75 31.75 0)
+    (property "Reference" "C2" (at 31.75 31.75 0)
       (effects (font (size 1.27 1.27)) (justify left))
     )
@@
       (effects (font (size 1.27 1.27)) (justify left))
     )
-    (property "Footprint" "" (at 28.9052 36.83 0)
+    (property "Footprint" "Capacitor_THT:C_Disc_D4.3mm_W1.9mm_P5.00mm" (at 28.9052 36.83 0)
       (effects (font (size 1.27 1.27)) hide)
     )
@@
       (project "555"
         (path "/ad638324-bd5b-4798-95cc-15159297f34d"
-          (reference "C1") (unit 1)
+          (reference "C2") (unit 1)
         )
       )
@@
       (effects (font (size 1.27 1.27)))
     )
-    (property "Footprint" "" (at 71.12 29.718 90)
+    (property "Footprint" "Resistor_THT:R_Axial_DIN0204_L3.6mm_D1.6mm_P2.54mm_Vertical" (at 71.12 29.718 90)
       (effects (font (size 1.27 1.27)) hide)
     )
@@
   (symbol (lib_id "Device:R") (at 66.04 64.77 180) (unit 1)
     (in_bom yes) (on_board yes) (dnp no)
-    (property "Reference" "R3" (at 63.5 64.77 90)
+    (property "Reference" "R1" (at 63.5 64.77 90)
       (effects (font (size 1.27 1.27)))
     )
@@
       (effects (font (size 1.27 1.27)))
     )
-    (property "Footprint" "" (at 67.818 64.77 90)
+    (property "Footprint" "Resistor_THT:R_Axial_DIN0204_L3.6mm_D1.6mm_P5.08mm_Horizontal" (at 67.818 64.77 90)
       (effects (font (size 1.27 1.27)) hide)
     )
@@
       (project "555"
         (path "/ad638324-bd5b-4798-95cc-15159297f34d"
-          (reference "R3") (unit 1)
+          (reference "R1") (unit 1)
         )
       )
@@
       (effects (font (size 1.27 1.27)))
     )
-    (property "Footprint" "OptoDevice:Vishay_CAST-3Pin" (at 45.72 42.545 0)
+    (property "Footprint" "Package_TO_SOT_THT:TO-92S_Wide" (at 45.72 42.545 0)
       (effects (font (size 1.27 1.27)) hide)
     )
@@
       (effects (font (size 1.27 1.27)) (justify left))
     )
-    (property "Footprint" "Package_SO:SOIC-8_3.9x4.9mm_P1.27mm" (at 62.23 85.09 0)
+    (property "Footprint" "Package_DIP:DIP-8_W7.62mm" (at 62.23 85.09 0)
       (effects (font (size 1.27 1.27)) hide)
     )
@@
       (effects (font (size 1.27 1.27)) (justify right))
     )
-    (property "Footprint" "" (at 80.01 78.74 0)
+    (property "Footprint" "LED_THT:LED_D5.0mm_Horizontal_O1.27mm_Z3.0mm" (at 80.01 78.74 0)
       (effects (font (size 1.27 1.27)) hide)
     )
@@
       (effects (font (size 1.27 1.27)) (justify left))
     )
-    (property "Footprint" "" (at 78.232 69.85 90)
+    (property "Footprint" "Resistor_THT:R_Axial_DIN0204_L3.6mm_D1.6mm_P2.54mm_Vertical" (at 78.232 69.85 90)
       (effects (font (size 1.27 1.27)) hide)
     )
@@
   (symbol (lib_id "Device:R") (at 71.12 33.02 90) (unit 1)
     (in_bom yes) (on_board yes) (dnp no)
-    (property "Reference" "R1" (at 71.12 30.48 90)
+    (property "Reference" "R3" (at 71.12 30.48 90)
       (effects (font (size 1.27 1.27)))
     )
@@
       (effects (font (size 1.27 1.27)))
     )
-    (property "Footprint" "" (at 71.12 34.798 90)
+    (property "Footprint" "Resistor_THT:R_Axial_DIN0204_L3.6mm_D1.6mm_P2.54mm_Vertical" (at 71.12 34.798 90)
       (effects (font (size 1.27 1.27)) hide)
     )
@@
       (project "555"
         (path "/ad638324-bd5b-4798-95cc-15159297f34d"
-          (reference "R1") (unit 1)
+          (reference "R3") (unit 1)
         )
       )
@@
   (symbol (lib_id "power:GND") (at 40.64 86.36 0) (unit 1)
     (in_bom yes) (on_board yes) (dnp no) (fields_autoplaced)
-    (property "Reference" "#PWR04" (at 40.64 92.71 0)
+    (property "Reference" "#PWR03" (at 40.64 92.71 0)
       (effects (font (size 1.27 1.27)) hide)
     )
@@
       (project "555"
         (path "/ad638324-bd5b-4798-95cc-15159297f34d"
-          (reference "#PWR04") (unit 1)
+          (reference "#PWR03") (unit 1)
         )
       )
@@
   (symbol (lib_id "power:+5V") (at 74.93 24.13 0) (unit 1)
     (in_bom yes) (on_board yes) (dnp no) (fields_autoplaced)
-    (property "Reference" "#PWR02" (at 74.93 27.94 0)
+    (property "Reference" "#PWR05" (at 74.93 27.94 0)
       (effects (font (size 1.27 1.27)) hide)
     )
@@
       (project "555"
         (path "/ad638324-bd5b-4798-95cc-15159297f34d"
-          (reference "#PWR02") (unit 1)
+          (reference "#PWR05") (unit 1)
         )
       )
@@
   (symbol (lib_id "power:GND") (at 25.4 102.87 0) (unit 1)
     (in_bom yes) (on_board yes) (dnp no) (fields_autoplaced)
-    (property "Reference" "#PWR03" (at 25.4 109.22 0)
+    (property "Reference" "#PWR01" (at 25.4 109.22 0)
       (effects (font (size 1.27 1.27)) hide)
     )
@@
       (project "555"
         (path "/ad638324-bd5b-4798-95cc-15159297f34d"
-          (reference "#PWR03") (unit 1)
+          (reference "#PWR01") (unit 1)
         )
       )
@@
   (symbol (lib_id "Device:C") (at 25.4 97.79 0) (unit 1)
     (in_bom yes) (on_board yes) (dnp no) (fields_autoplaced)
-    (property "Reference" "C2" (at 29.21 96.52 0)
+    (property "Reference" "C1" (at 29.21 96.52 0)
       (effects (font (size 1.27 1.27)) (justify left))
     )
@@
       (effects (font (size 1.27 1.27)) (justify left))
     )
-    (property "Footprint" "" (at 26.3652 101.6 0)
+    (property "Footprint" "Capacitor_THT:C_Disc_D4.3mm_W1.9mm_P5.00mm" (at 26.3652 101.6 0)
       (effects (font (size 1.27 1.27)) hide)
     )
@@
       (project "555"
         (path "/ad638324-bd5b-4798-95cc-15159297f34d"
-          (reference "C2") (unit 1)
+          (reference "C1") (unit 1)
         )
       )
@@
       (effects (font (size 1.27 1.27)) (justify right))
     )
-    (property "Footprint" "" (at 66.04 80.01 0)
+    (property "Footprint" "Potentiometer_THT:Potentiometer_Bourns_3296W_Vertical" (at 66.04 80.01 0)
       (effects (font (size 1.27 1.27)) hide)
     )
@@
   (symbol (lib_id "power:GND") (at 57.15 44.45 0) (unit 1)
     (in_bom yes) (on_board yes) (dnp no) (fields_autoplaced)
-    (property "Reference" "#PWR01" (at 57.15 50.8 0)
+    (property "Reference" "#PWR04" (at 57.15 50.8 0)
       (effects (font (size 1.27 1.27)) hide)
     )
@@
       (project "555"
         (path "/ad638324-bd5b-4798-95cc-15159297f34d"
-          (reference "#PWR01") (unit 1)
+          (reference "#PWR04") (unit 1)
         )
       )
@@
   (symbol (lib_id "power:+5V") (at 80.01 64.77 0) (unit 1)
     (in_bom yes) (on_board yes) (dnp no) (fields_autoplaced)
-    (property "Reference" "#PWR05" (at 80.01 68.58 0)
+    (property "Reference" "#PWR06" (at 80.01 68.58 0)
       (effects (font (size 1.27 1.27)) hide)
     )
@@
       (project "555"
         (path "/ad638324-bd5b-4798-95cc-15159297f34d"
-          (reference "#PWR05") (unit 1)
+          (reference "#PWR06") (unit 1)
         )
       )
@@
   (symbol (lib_id "power:+5V") (at 40.64 64.77 0) (unit 1)
     (in_bom yes) (on_board yes) (dnp no) (fields_autoplaced)
-    (property "Reference" "#PWR06" (at 40.64 68.58 0)
+    (property "Reference" "#PWR02" (at 40.64 68.58 0)
       (effects (font (size 1.27 1.27)) hide)
     )
@@
       (project "555"
         (path "/ad638324-bd5b-4798-95cc-15159297f34d"
-          (reference "#PWR06") (unit 1)
-        )
-      )
+          (reference "#PWR02") (unit 1)
+        )
+      )

Commit message: arranque PCB 555 falta rutear
Parts:
- R2, R3, R4: footprint Resistor_THT:R_Axial_DIN0204_L3.6mm_D1.6mm_P2.54mm_Vertical -> Resistor_THT:R_Axial_DIN0204_L3.6mm_D1.6mm_P5.08mm_Horizontal
Connections:
- net GND: now also U2.2 (Vs); no longer U2.1 (GND)
- net at C2.1, R2.1: now also U2.1 (GND); no longer U2.2 (Vs)
Changed lines of the file:
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@@
   (junction (at 66.04 74.93) (diameter 0) (color 0 0 0 0)
   )
+  (junction (at 66.04 33.02) (diameter 0) (color 0 0 0 0)
+  )
   (junction (at 66.04 85.09) (diameter 0) (color 0 0 0 0)
   )
+  (junction (at 53.34 85.09) (diameter 0) (color 0 0 0 0)
+  )
+  (junction (at 58.42 24.13) (diameter 0) (color 0 0 0 0)
+  )
   (junction (at 57.15 41.91) (diameter 0) (color 0 0 0 0)
   )
-  (junction (at 53.34 85.09) (diameter 0) (color 0 0 0 0)
-  )
-  (junction (at 63.5 27.94) (diameter 0) (color 0 0 0 0)
-  )
-  (junction (at 66.04 33.02) (diameter 0) (color 0 0 0 0)
-  )
   (wire (pts (xy 53.34 80.01) (xy 53.34 85.09))
     (stroke (width 0) (type default))
@@
     (stroke (width 0) (type default))
   )
-  (wire (pts (xy 57.15 38.1) (xy 57.15 41.91))
-    (stroke (width 0) (type default))
-  )
   (wire (pts (xy 27.94 41.91) (xy 27.94 36.83))
     (stroke (width 0) (type default))
   )
+  (wire (pts (xy 60.96 27.94) (xy 60.96 41.91))
+    (stroke (width 0) (type default))
+  )
   (wire (pts (xy 63.5 24.13) (xy 63.5 27.94))
     (stroke (width 0) (type default))
   )
-  (wire (pts (xy 63.5 24.13) (xy 27.94 24.13))
+  (wire (pts (xy 63.5 24.13) (xy 58.42 24.13))
     (stroke (width 0) (type default))
   )
@@
     (stroke (width 0) (type default))
   )
+  (wire (pts (xy 57.15 33.02) (xy 66.04 33.02))
+    (stroke (width 0) (type default))
+  )
   (wire (pts (xy 53.34 69.85) (xy 73.66 69.85))
     (stroke (width 0) (type default))
@@
     (stroke (width 0) (type default))
   )
+  (wire (pts (xy 58.42 24.13) (xy 27.94 24.13))
+    (stroke (width 0) (type default))
+  )
   (wire (pts (xy 40.64 86.36) (xy 40.64 85.09))
     (stroke (width 0) (type default))
@@
     (stroke (width 0) (type default))
   )
+  (wire (pts (xy 57.15 38.1) (xy 58.42 38.1))
+    (stroke (width 0) (type default))
+  )
   (wire (pts (xy 25.4 69.85) (xy 27.94 69.85))
     (stroke (width 0) (type default))
@@
     (stroke (width 0) (type default))
   )
-  (wire (pts (xy 57.15 33.02) (xy 66.04 33.02))
-    (stroke (width 0) (type default))
-  )
   (wire (pts (xy 66.04 68.58) (xy 66.04 74.93))
     (stroke (width 0) (type default))
@@
     (stroke (width 0) (type default))
   )
+  (wire (pts (xy 57.15 27.94) (xy 60.96 27.94))
+    (stroke (width 0) (type default))
+  )
+  (wire (pts (xy 58.42 24.13) (xy 58.42 38.1))
+    (stroke (width 0) (type default))
+  )
   (wire (pts (xy 57.15 44.45) (xy 57.15 41.91))
     (stroke (width 0) (type default))
   )
-  (wire (pts (xy 57.15 27.94) (xy 63.5 27.94))
-    (stroke (width 0) (type default))
-  )
   (wire (pts (xy 66.04 76.2) (xy 66.04 74.93))
+    (stroke (width 0) (type default))
+  )
+  (wire (pts (xy 60.96 41.91) (xy 57.15 41.91))
     (stroke (width 0) (type default))
   )
@@
       (effects (font (size 1.27 1.27)) hide)
     )
-    (pin "2")
-    (pin "1")
+    (pin "1")
+    (pin "2")
     (instances
       (project "555"
@@
       (effects (font (size 1.27 1.27)))
     )
-    (property "Footprint" "Resistor_THT:R_Axial_DIN0204_L3.6mm_D1.6mm_P2.54mm_Vertical" (at 71.12 29.718 90)
+    (property "Footprint" "Resistor_THT:R_Axial_DIN0204_L3.6mm_D1.6mm_P5.08mm_Horizontal" (at 71.12 29.718 90)
       (effects (font (size 1.27 1.27)) hide)
     )
@@
       (effects (font (size 1.27 1.27)) hide)
     )
+    (pin "1")
     (pin "8")
-    (pin "1")
     (pin "2")
     (pin "3")
     (pin "4")
+    (pin "5")
+    (pin "6")
     (pin "7")
-    (pin "6")
-    (pin "5")
     (instances
       (project "555"
@@
       (effects (font (size 1.27 1.27)) (justify left))
     )
-    (property "Footprint" "Resistor_THT:R_Axial_DIN0204_L3.6mm_D1.6mm_P2.54mm_Vertical" (at 78.232 69.85 90)
+    (property "Footprint" "Resistor_THT:R_Axial_DIN0204_L3.6mm_D1.6mm_P5.08mm_Horizontal" (at 78.232 69.85 90)
       (effects (font (size 1.27 1.27)) hide)
     )
@@
       (effects (font (size 1.27 1.27)))
     )
-    (property "Footprint" "Resistor_THT:R_Axial_DIN0204_L3.6mm_D1.6mm_P2.54mm_Vertical" (at 71.12 34.798 90)
+    (property "Footprint" "Resistor_THT:R_Axial_DIN0204_L3.6mm_D1.6mm_P5.08mm_Horizontal" (at 71.12 34.798 90)
       (effects (font (size 1.27 1.27)) hide)
     )
@@
       (effects (font (size 1.27 1.27)) hide)
     )
-    (pin "2")
-    (pin "1")
+    (pin "1")
+    (pin "2")
     (instances
       (project "555"
@@
       (effects (font (size 1.27 1.27)) hide)
     )
+    (pin "1")
+    (pin "2")
     (pin "3")
-    (pin "1")
-    (pin "2")
-    (instances
-      (project "555"
+    (instances
+      (project "555"

Commit message: ana
Parts:
- removed R3: 22k, Resistor_THT:R_Axial_DIN0204_L3.6mm_D1.6mm_P5.08mm_Horizontal, symbol Device:R
- added J1: Conn_01x03_Pin, Connector_PinHeader_2.54mm:PinHeader_1x03_P2.54mm_Vertical, symbol Connector:Conn_01x03_Pin
Connections:
- net +5V: now also R1.2, U1.4 (R), J1.1 (Pin_1)
- net GND: now also J1.2 (Pin_2)
- net Sensores: now also J1.3 (Pin_3)
Changed lines of the file:
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@@
   (junction (at 25.4 92.71) (diameter 0) (color 0 0 0 0)
   )
-  (junction (at 74.93 27.94) (diameter 0) (color 0 0 0 0)
-  )
   (junction (at 66.04 74.93) (diameter 0) (color 0 0 0 0)
   )
@@
   (junction (at 58.42 24.13) (diameter 0) (color 0 0 0 0)
   )
+  (junction (at 40.64 57.15) (diameter 0) (color 0 0 0 0)
+  )
   (junction (at 57.15 41.91) (diameter 0) (color 0 0 0 0)
   )
@@
     (stroke (width 0) (type default))
   )
+  (wire (pts (xy 94.615 52.07) (xy 99.695 52.07))
+    (stroke (width 0) (type default))
+  )
+  (wire (pts (xy 95.25 59.055) (xy 94.615 59.055))
+    (stroke (width 0) (type default))
+  )
   (wire (pts (xy 63.5 24.13) (xy 58.42 24.13))
     (stroke (width 0) (type default))
@@
     (stroke (width 0) (type default))
   )
+  (wire (pts (xy 94.615 59.055) (xy 94.615 54.61))
+    (stroke (width 0) (type default))
+  )
   (wire (pts (xy 74.93 24.13) (xy 74.93 27.94))
     (stroke (width 0) (type default))
@@
     (stroke (width 0) (type default))
   )
+  (wire (pts (xy 100.33 49.53) (xy 94.615 49.53))
+    (stroke (width 0) (type default))
+  )
   (wire (pts (xy 58.42 24.13) (xy 27.94 24.13))
     (stroke (width 0) (type default))
@@
     (stroke (width 0) (type default))
   )
+  (wire (pts (xy 40.64 56.515) (xy 40.64 57.15))
+    (stroke (width 0) (type default))
+  )
   (wire (pts (xy 25.4 69.85) (xy 27.94 69.85))
     (stroke (width 0) (type default))
@@
     (stroke (width 0) (type default))
   )
-  (wire (pts (xy 74.93 27.94) (xy 74.93 33.02))
+  (wire (pts (xy 40.64 57.15) (xy 40.64 64.77))
     (stroke (width 0) (type default))
   )
@@
     (stroke (width 0) (type default))
   )
+  (wire (pts (xy 40.64 57.15) (xy 66.04 57.15))
+    (stroke (width 0) (type default))
+  )
   (wire (pts (xy 57.15 27.94) (xy 60.96 27.94))
     (stroke (width 0) (type default))
@@
     (stroke (width 0) (type default))
   )
-  (wire (pts (xy 22.86 57.15) (xy 66.04 57.15))
-    (stroke (width 0) (type default))
+  (wire (pts (xy 22.86 57.15) (xy 40.64 57.15))
+    (stroke (width 0) (type default))
+  )
+  (global_label "Sensores" (shape input) (at 95.25 59.055 0) (fields_autoplaced)
+    (effects (font (size 1.27 1.27)) (justify left))
+    (property "Intersheetrefs" "${INTERSHEET_REFS}" (at 106.7623 59.055 0)
+      (effects (font (size 1.27 1.27)) (justify left) hide)
+    )
   )
   (global_label "Sensores" (shape input) (at 66.04 41.91 0) (fields_autoplaced)
@@
     )
   )
+  (symbol (lib_id "Connector:Conn_01x03_Pin") (at 89.535 52.07 0) (unit 1)
+    (in_bom yes) (on_board yes) (dnp no) (fields_autoplaced)
+    (property "Reference" "J1" (at 90.17 45.72 0)
+      (effects (font (size 1.27 1.27)))
+    )
+    (property "Value" "Conn_01x03_Pin" (at 90.17 48.26 0)
+      (effects (font (size 1.27 1.27)))
+    )
+    (property "Footprint" "Connector_PinHeader_2.54mm:PinHeader_1x03_P2.54mm_Vertical" (at 89.535 52.07 0)
+      (effects (font (size 1.27 1.27)) hide)
+    )
+    (property "Datasheet" "~" (at 89.535 52.07 0)
+      (effects (font (size 1.27 1.27)) hide)
+    )
+    (pin "1")
+    (pin "2")
+    (pin "3")
+    (instances
+      (project "555"
+        (path "/ad638324-bd5b-4798-95cc-15159297f34d"
+          (reference "J1") (unit 1)
+        )
+      )
+    )
+  )
+  (symbol (lib_id "power:GND") (at 99.695 52.07 0) (unit 1)
+    (in_bom yes) (on_board yes) (dnp no)
+    (property "Reference" "#PWR08" (at 99.695 58.42 0)
+      (effects (font (size 1.27 1.27)) hide)
+    )
+    (property "Value" "GND" (at 99.695 55.88 0)
+      (effects (font (size 1.27 1.27)))
+    )
+    (property "Footprint" "" (at 99.695 52.07 0)
+      (effects (font (size 1.27 1.27)) hide)
+    )
+    (property "Datasheet" "" (at 99.695 52.07 0)
+      (effects (font (size 1.27 1.27)) hide)
+    )
+    (pin "1")
+    (instances
+      (project "555"
+        (path "/ad638324-bd5b-4798-95cc-15159297f34d"
+          (reference "#PWR08") (unit 1)
+        )
+      )
+    )
+  )
   (symbol (lib_id "Device:C") (at 27.94 33.02 0) (unit 1)
     (in_bom yes) (on_board yes) (dnp no) (fields_autoplaced)
@@
         (path "/ad638324-bd5b-4798-95cc-15159297f34d"
           (reference "R1") (unit 1)
+        )
+      )
+    )
+  )
+  (symbol (lib_id "power:+5V") (at 100.33 49.53 0) (unit 1)
+    (in_bom yes) (on_board yes) (dnp no) (fields_autoplaced)
+    (property "Reference" "#PWR07" (at 100.33 53.34 0)
+      (effects (font (size 1.27 1.27)) hide)
+    )
+    (property "Value" "+5V" (at 100.33 45.72 0)
+      (effects (font (size 1.27 1.27)))
+    )
+    (property "Footprint" "" (at 100.33 49.53 0)
+      (effects (font (size 1.27 1.27)) hide)
+    )
+    (property "Datasheet" "" (at 100.33 49.53 0)
+      (effects (font (size 1.27 1.27)) hide)
+    )
+    (pin "1")
+    (instances
+      (project "555"
+        (path "/ad638324-bd5b-4798-95cc-15159297f34d"
+          (reference "#PWR07") (unit 1)
         )
       )
@@
     )
   )
-  (symbol (lib_id "Device:R") (at 71.12 33.02 90) (unit 1)
-    (in_bom yes) (on_board yes) (dnp no)
-    (property "Reference" "R3" (at 71.12 30.48 90)
-      (effects (font (size 1.27 1.27)))
-    )
-    (property "Value" "22k" (at 71.12 33.02 90)
-      (effects (font (size 1.27 1.27)))
-    )
-    (property "Footprint" "Resistor_THT:R_Axial_DIN0204_L3.6mm_D1.6mm_P5.08mm_Horizontal" (at 71.12 34.798 90)
-      (effects (font (size 1.27 1.27)) hide)
-    )
-    (property "Datasheet" "~" (at 71.12 33.02 0)
-      (effects (font (size 1.27 1.27)) hide)
-    )
-    (pin "1")
-    (pin "2")
-    (instances
-      (project "555"
-        (path "/ad638324-bd5b-4798-95cc-15159297f34d"
-          (reference "R3") (unit 1)
-        )
-      )
-    )
-  )
   (symbol (lib_id "power:GND") (at 40.64 86.36 0) (unit 1)
     (in_bom yes) (on_board yes) (dnp no) (fields_autoplaced)
@@
     )
   )
-  (symbol (lib_id "power:+5V") (at 40.64 64.77 0) (unit 1)
-    (in_bom yes) (on_board yes) (dnp no) (fields_autoplaced)
-    (property "Reference" "#PWR02" (at 40.64 68.58 0)
-      (effects (font (size 1.27 1.27)) hide)
-    )
-    (property "Value" "+5V" (at 40.64 59.69 0)
-      (effects (font (size 1.27 1.27)))
-    )
-    (property "Footprint" "" (at 40.64 64.77 0)
-      (effects (font (size 1.27 1.27)) hide)
-    )
-    (property "Datasheet" "" (at 40.64 64.77 0)
-      (effects (font (size 1.27 1.27)) hide)
-    )
+  (symbol (lib_id "power:+5V") (at 40.64 56.515 0) (unit 1)
+    (in_bom yes) (on_board yes) (dnp no) (fields_autoplaced)
+    (property "Reference" "#PWR02" (at 40.64 60.325 0)
+      (effects (font (size 1.27 1.27)) hide)
+    )
+    (property "Value" "+5V" (at 40.64 51.435 0)
+      (effects (font (size 1.27 1.27)))
+    )
+    (property "Footprint" "" (at 40.64 56.515 0)
+      (effects (font (size 1.27 1.27)) hide)
+    )
+    (property "Datasheet" "" (at 40.64 56.515 0)
+      (effects (font (size 1.27 1.27)) hide)
+    )
