File: 555/555.kicad_sch (KiCad schematic)
At the start: 10 parts, among them J1 Conn_01x03_Pin, U1 LM555xM, U2 TSOP17xx

Commit message: lalalalal
Parts:
- removed J1: Conn_01x03_Pin, Connector_PinHeader_2.54mm:PinHeader_1x03_P2.54mm_Vertical, symbol Connector:Conn_01x03_Pin
- added C3, C4: 104, Capacitor_THT:C_Disc_D4.3mm_W1.9mm_P5.00mm, symbol Device:C
- added D2, D3: LED, LED_THT:LED_D5.0mm_Horizontal_O1.27mm_Z3.0mm, symbol Device:LED
- added J1: Conn_02x05_Counter_Clockwise, Connector_IDC:IDC-Header_2x05_P2.54mm_Horizontal, symbol Connector_Generic:Conn_02x05_Counter_Clockwise
- added Q1: BC547, Package_TO_SOT_THT:TO-92_Wide, symbol Transistor_BJT:BC547
- added R3: 4.7k, Resistor_SMD:R_1206_3216Metric_Pad1.30x1.75mm_HandSolder, symbol Device:R
- added R5, R8: 100, Resistor_SMD:R_1206_3216Metric_Pad1.30x1.75mm_HandSolder, symbol Device:R
- added R6, R7: 100, Resistor_THT:R_Axial_DIN0207_L6.3mm_D2.5mm_P10.16mm_Horizontal, symbol Device:R
- added U3, U4: TSOP17xx, Package_TO_SOT_THT:TO-92S_Wide, symbol Interface_Optical:TSOP17xx
- R1, R2: footprint Resistor_THT:R_Axial_DIN0204_L3.6mm_D1.6mm_P5.08mm_Horizontal -> Resistor_SMD:R_1206_3216Metric_Pad1.30x1.75mm_HandSolder
- R4: footprint Resistor_THT:R_Axial_DIN0204_L3.6mm_D1.6mm_P5.08mm_Horizontal -> Resistor_THT:R_Axial_DIN0207_L6.3mm_D2.5mm_P10.16mm_Horizontal
Connections:
- net +5V: now also J1.2 (Pin_2), R5.2, R6.1, R7.1, R8.2
- net GND: now also C3.2, C4.2, J1.7 (Pin_7), Q1.1 (C), U3.2 (Vs), U4.2 (Vs)
- net Sensores: now also J1.9 (Pin_9)
- net at U1.3 (Q): now also R3.1; no longer D1.1 (K)
- new net: D2.2 (A), R6.2
- new net: Q1.2 (B), R3.2
- new net: C4.1, R8.1, U4.1 (GND)
- new net: C3.1, R5.1, U3.1 (GND)
- new net: D3.2 (A), R7.2
- new net 38khz: D1.1 (K), D2.1 (K), D3.1 (K), Q1.3 (E)
- new net Sensores_2: J1.1 (Pin_1), U3.3 (OUT)
- new net Sensores_3: J1.5 (Pin_5), U4.3 (OUT)
Other:
- moved on the sheet: C2

Commit message: soporte tof
Parts:
- R4: footprint Resistor_THT:R_Axial_DIN0207_L6.3mm_D2.5mm_P10.16mm_Horizontal -> Resistor_SMD:R_1206_3216Metric_Pad1.30x1.75mm_HandSolder
Changed lines of the file:
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@@
       (effects (font (size 1.27 1.27)) (justify left))
     )
-    (property "Footprint" "Resistor_THT:R_Axial_DIN0207_L6.3mm_D2.5mm_P10.16mm_Horizontal" (at 78.232 69.85 90)
+    (property "Footprint" "Resistor_SMD:R_1206_3216Metric_Pad1.30x1.75mm_HandSolder" (at 78.232 69.85 90)
       (effects (font (size 1.27 1.27)) hide)
     )
