File: atemga/atmega.kicad_pcb (KiCad board)
At the start: 2 copper layers, 182.8 x 33.6 mm, 24 parts, among them J1 Conn_02x05_Counter_Clockwise, Q1 BC547, U1 LM555xM, U2 TSOP17xx, U3 TSOP17xx, U4 TSOP17xx

Commit message: pdf atemga
Parts:
- removed RV1: pote, Potentiometer_THT:Potentiometer_Bourns_3296W_Vertical
- added C5: C, Capacitor_SMD:C_1206_3216Metric_Pad1.33x1.80mm_HandSolder, B.Cu at (78.7, 36.5)
- added Y1: Crystal, Crystal:Crystal_HC18-U_Vertical, F.Cu at (70.7, 35.6)
- C1: value 102 -> C; footprint Capacitor_THT:C_Disc_D4.3mm_W1.9mm_P5.00mm -> Capacitor_SMD:C_1206_3216Metric_Pad1.33x1.80mm_HandSolder; moved to B.Cu
- R1: value 1k8 -> 100
- U1: value LM555xM -> ATmega328-P; footprint Package_DIP:DIP-8_W7.62mm -> Package_DIP:DIP-28_W7.62mm
- moved C1 22.0 mm to (76.3, 43.6)
- moved R3 19.1 mm to (107.8, 40.5), turned to 0 degrees
- moved R1 16.8 mm to (83.1, 43.5), turned to 180 degrees
- moved U1 3.35 mm to (96.5, 40.6)
- moved J1 1.51 mm to (167.8, 42.3)
- moved R7 1.44 mm to (200.5, 51.5)
- moved R5 1.38 mm to (193.8, 48.2)
- moved C4 1.31 mm to (51.7, 49.1)
- moved C3 1.03 mm to (195.2, 43.7)
- moved R6 0.35 mm to (47.2, 49.1)
Connections:
- C1 pad 1: Net-(U1-THR) -> Net-(U1-XTAL2/PB7)
- R1 pad 1: Net-(U1-DIS) -> Net-(U1-~{RESET}/PC6)
- R3 pad 1: Net-(U1-Q) -> Net-(U1-PB3)
- U1 pad 1: GND -> Net-(U1-~{RESET}/PC6)
- U1 pad 2: Net-(U1-THR) -> unconnected-(U1-PD0-Pad2)
- U1 pad 3: Net-(U1-Q) -> unconnected-(U1-PD1-Pad3)
- U1 pad 4: +5V -> unconnected-(U1-PD2-Pad4)
- U1 pad 6: Net-(U1-THR) -> unconnected-(U1-PD4-Pad6)
- U1 pad 7: Net-(U1-DIS) -> +5V
- U1 pad 8: +5V -> GND
Routing:
- net Net-(U1-PB3): track 0.00 -> 67.3 mm
- net Net-(U1-THR): track 51.0 -> 0.00 mm
- net GND: track 383.8 -> 431.9 mm
- net +5V: track 265.8 -> 229.8 mm, vias 4 -> 2
- net Net-(Q1-B): track 36.2 -> 4.39 mm
- net Net-(U1-DIS): track 30.8 -> 0.00 mm
- net Net-(U1-~{RESET}/PC6): track 0.00 -> 14.0 mm
- net Net-(U1-XTAL2/PB7): track 0.00 -> 10.2 mm
- net Net-(U1-XTAL1/PB6): track 0.00 -> 8.67 mm
- net Net-(U1-Q): track 7.68 -> 0.00 mm
- net Sensores_3: track 122.1 -> 125.7 mm
- net Net-(U3-GND): track 11.3 -> 8.65 mm
- net Sensores_2: track 49.2 -> 51.5 mm
- net 38khz: track 198.9 -> 200.8 mm
- net Net-(D1-A): track 28.8 -> 27.8 mm
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