File: PCB/vulcano v1/vulcano v1.kicad_sch (KiCad schematic)
At the start: 11 parts, among them J1 Screw_Terminal_01x02, J2 Screw_Terminal_01x02, J3 conector t, U1 DOIT-ESP32-DEVKIT-V1, U2 LM7809_TO220, U3 LM7806_TO220

Commit message: placa principal
Parts:
- added A1: Arduino_UNO_R2, Module:Arduino_UNO_R2, symbol MCU_Module:Arduino_UNO_R2
- added J4: Conn_02x05_Counter_Clockwise, Connector_IDC:IDC-Header_2x05_P2.54mm_Vertical, symbol Connector_Generic:Conn_02x05_Counter_Clockwise
- added J5, J6: Conn_01x05_Pin, Connector_PinSocket_2.54mm:PinSocket_1x05_P2.54mm_Vertical, symbol Connector:Conn_01x05_Pin
- added J7, J8: Conn_01x06_Pin, Connector_PinSocket_2.54mm:PinSocket_1x06_P2.54mm_Vertical, symbol Connector:Conn_01x06_Pin
- added Q1, Q2, Q3, Q4, Q5: BC547, Package_TO_SOT_THT:TO-92_Wide, symbol Transistor_BJT:BC547
- added R12, R15, R3, R6, R9: 4k7, Resistor_THT:R_Axial_DIN0204_L3.6mm_D1.6mm_P7.62mm_Horizontal, symbol Device:R
- added SW1: SW_SPDT, Button_Switch_THT:SW_CuK_JS202011CQN_DPDT_Straight, symbol Switch:SW_SPDT
- C1, C2, C3, C4: footprint (none) -> Capacitor_THT:C_Disc_D4.3mm_W1.9mm_P5.00mm
- J1: footprint Connector_AMASS:AMASS_XT60-F_1x02_P7.20mm_Vertical -> TerminalBlock:TerminalBlock_bornier-2_P5.08mm
- J3: value conector t -> Screw_Terminal_01x02; footprint Connector_AMASS:AMASS_XT60-F_1x02_P7.20mm_Vertical -> TerminalBlock:TerminalBlock_bornier-2_P5.08mm
Connections:
- net +12V: now also SW1.1 (A)
- net GND: now also J2.2 (Pin_2), U1.17 (GND), A1.6 (GND), A1.7 (GND), J4.7 (Pin_7), J5.4 (Pin_4), J6.4 (Pin_4), J7.5 (Pin_5), J8.5 (Pin_5); no longer J1.1 (Pin_1)
- net VCC: now also SW1.2 (B); no longer J2.2 (Pin_2)
- net PWMA: now reaches U1.10 (GPIO27_ADC2-CH7_RTC-GPIO17)
- net PWMA: now also A1.20 (D5)
- net BIN1: now reaches U1.11 (GPIO14_ADC2-CH6_HSPI-CLK_RTC-GPIO16)
- net BIN1: now also A1.19 (D4)
- net +5V: now reaches U1.18 (VIN)
- net +5V: now also D1.1 (K), A1.5 (+5V), J4.2 (Pin_2), J7.1 (Pin_1), J8.1 (Pin_1)
- net +3.3V: now reaches U1.19 (3V3)
- net +3.3V: now also J5.5 (Pin_5), J6.5 (Pin_5), Q1.1 (C), Q2.1 (C), Q3.1 (C), Q4.1 (C), Q5.1 (C)
- net X_SHUT_2: now reaches U1.20 (GPIO6_SCK/CLK)
- net X_SHUT_2: now also J5.1 (Pin_1)
- net X_SHUT_1: now reaches U1.21 (GPIO7_SDO/SD0)
- net X_SHUT_1: now also J6.1 (Pin_1)
- net SENSOR_5_PIN: now reaches U1.26 (GPIO4_ADC2-CH0_RTC-GPIO10)
- net SENSOR_5_PIN: now also Q5.3 (E)
- net SENSOR_2_PIN: now reaches U1.29 (GPIO5_VSPI-CS0)
- net SENSOR_2_PIN: now also Q2.3 (E)
- net SENSOR_1_PIN: now reaches U1.30 (GPIO18_VSPI-CLK)
- net SENSOR_1_PIN: now also Q1.3 (E)
- net SENSOR_3_PIN: now reaches U1.31 (GPIO19_VSPI-MISO)
- net SENSOR_3_PIN: now also Q3.3 (E)
- net SDA: now reaches U1.32 (GPIO21_I2C-SDA)
- net SDA: now also J5.2 (Pin_2), J6.2 (Pin_2)
- net SCL: now reaches U1.35 (GPIO22_I2C-SCL)
- net SCL: now also J5.3 (Pin_3), J6.3 (Pin_3)
- net SENSOR_4_PIN: now reaches U1.36 (GPIO23_VSPI-MOSI)
- net SENSOR_4_PIN: now also Q4.3 (E)
- net BIN2: now reaches U1.6 (GPIO32_ADC1-CH4_RTC-GPIO9)
- net BIN2: now also A1.24 (D9)
- net AIN2: now reaches U1.7 (GPIO33_ADC1-CH5_RTC-GPIO8)
- net AIN2: now also A1.23 (D8)
- net AIN1: now reaches U1.8 (GPIO25_ADC2-CH8_DAC1_RTC-GPIO6)
- net AIN1: now also A1.22 (D7)
- net PWMB: now reaches U1.9 (GPIO26_ADC2-CH9_DAC2_RTC-GPIO7)
- net PWMB: now also A1.21 (D6)
- new net: Q5.2 (B), R15.2
- new net: Q3.2 (B), R9.2
- new net: Q4.2 (B), R12.2
- new net: Q2.2 (B), R6.2
- new net: J1.1 (Pin_1), SW1.3 (C)
- new net: Q1.2 (B), R3.2
- new net 38KHZ: J4.10 (Pin_10), J7.6 (Pin_6), J8.6 (Pin_6)
- new net RX: J7.4 (Pin_4), R12.1
- new net RX_1: J8.4 (Pin_4), R15.1
- new net Sensores: J4.5 (Pin_5), R3.1
- new net Sensores_2: J4.9 (Pin_9), R6.1
- new net Sensores_3: J4.1 (Pin_1), R9.1

Commit message: pcb vulcano terminada (reviasala ana)
Parts:
- removed SW1: SW_SPDT, Button_Switch_THT:SW_CuK_JS202011CQN_DPDT_Straight, symbol Switch:SW_SPDT
- added BZ1: Buzzer, Buzzer_Beeper:MagneticBuzzer_Kingstate_KCG0601, symbol Device:Buzzer
- added C5: C_Polarized_US, Capacitor_THT:CP_Radial_D8.0mm_P5.00mm, symbol Device:C_Polarized_US
- added J10: Conn_01x03_Pin, Connector_PinHeader_2.54mm:PinHeader_1x03_P2.54mm_Vertical, symbol Connector:Conn_01x03_Pin
- added J2: Conn_01x06_Pin, Connector_PinHeader_2.54mm:PinHeader_1x06_P2.54mm_Vertical, symbol Connector:Conn_01x06_Pin
- added J9: Conn_01x05_Pin, Connector_PinHeader_2.54mm:PinHeader_1x05_P2.54mm_Vertical, symbol Connector:Conn_01x05_Pin
- added Q6: BC547, Package_TO_SOT_THT:TO-92_Wide, symbol Transistor_BJT:BC547
- added R1, R2: 4k7, Resistor_THT:R_Axial_DIN0204_L3.6mm_D1.6mm_P7.62mm_Horizontal, symbol Device:R
- added SW2: SW_Push, Button_Switch_THT:SW_PUSH_6mm, symbol Switch:SW_Push
- J1, J3: footprint TerminalBlock:TerminalBlock_bornier-2_P5.08mm -> deans:DEANS
- J2: footprint Connector_AMASS:AMASS_XT60-F_1x02_P7.20mm_Vertical -> Connector_AMASS:AMASS_XT60-M_1x02_P7.20mm_Vertical
Connections:
- net +3.3V: now also A1.5 (+5V), J2.6 (Pin_6), J9.2 (Pin_2), R1.2
- net +5V: now also J10.2 (Pin_2), Q6.1 (C); no longer A1.5 (+5V)
- net GND: now also BZ1.2 (+), C5.2, J10.3 (Pin_3), J2.5 (Pin_5), J9.1 (Pin_1), SW2.1
- net VCC: now also J1.1 (Pin_1), C5.1
- net X_SHUT_2: now also U1.22 (GPIO8_SDI/SD1); no longer U1.20 (GPIO6_SCK/CLK)
- net DI: now reaches U1.13 (GPIO13_ADC2-CH4_HSPI-MOSI_RTC-GPIO14)
- net DI: now also J10.1 (Pin_1)
- net SW: now reaches U1.14 (GPIO9_SHD/SD2)
- net SW: now also J9.3 (Pin_3)
- net DT: now reaches U1.15 (GPIO10_SWP/SD3)
- net DT: now also J9.4 (Pin_4)
- net CLK: now reaches U1.16 (GPIO11_CSC/CMD)
- net CLK: now also J9.5 (Pin_5)
- net CNY_1: now reaches U1.2 (GPIO36_ADC-CH0_SENS-VP_RTC-GPIO0)
- net CNY_1: now also J2.1 (Pin_1)
- net CNY_4: now reaches U1.25 (GPIO2_ADC2-CH2_RTC-GPIO12)
- net CNY_4: now also J2.4 (Pin_4)
- net buzzer: now reaches U1.28 (GPIO17_UART2-TX)
- net buzzer: now also R2.1
- net CNY_2: now reaches U1.3 (GPIO39_ADC1-CH3_SENS-VN_RTC-GPIO3)
- net CNY_2: now also J2.2 (Pin_2)
- net CNY_3: now reaches U1.4 (GPIO34_ADC1-CH6_RTC-GPIO4)
- net CNY_3: now also J2.3 (Pin_3)
- net INIT: now reaches U1.5 (GPIO35_ADC1-CH7_RTC-GPIO5)
- net INIT: now also R1.1, SW2.2
- new net: Q6.2 (B), R2.2
- new net: BZ1.1 (-), Q6.3 (E)

Commit message: placa central lista
Parts:
- C5: footprint Capacitor_THT:CP_Radial_D8.0mm_P5.00mm -> Capacitor_THT:CP_Radial_D13.0mm_P5.00mm
Changed lines of the file:
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@@
       (effects (font (size 1.27 1.27)) (justify left))
     )
-    (property "Footprint" "Capacitor_THT:CP_Radial_D8.0mm_P5.00mm" (at 76.835 34.29 0)
+    (property "Footprint" "Capacitor_THT:CP_Radial_D13.0mm_P5.00mm" (at 76.835 34.29 0)
       (effects (font (size 1.27 1.27)) hide)
     )
